File: swift-nav.sch (EAGLE design)
At the start: 111 parts, among them J1 SMA, J3 SMA, J4 PIN_HDR_EDG_1.27MM_5-2, J6 ZX62-B-5PA, U1 6SLX9FTG256, U10 MAX2769, U12 PT7M8206B33TA5EX, U13 M25PX80, U2 LTC3407A, U3 STM32-M-64-LQFP, U4 7Q-16.368MBG-T, U8 B4050, X3 FPGA_DEBUG_HDR

Commit message: Starting layout
Parts:
- removed C2: 0R, rcl:C-EUC0402
Connections:
- removed net N$29: C2.1, U10_ANA.LNA_IN1
- net N$11: now also U10_ANA.LNA_IN1; no longer C2.2
Other:
- note removed: "50 ohm lines"
- moved on the sheet: ANT1
Changed lines of the file:
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@@
 <setting verticaltext="up"/>
 </settings>
-<grid distance="0.1" unitdist="inch" unit="inch" style="lines" multiple="1" display="no" altdistance="0.01" altunitdist="inch" altunit="inch"/>
+<grid distance="0.025" unitdist="inch" unit="inch" style="lines" multiple="1" display="yes" altdistance="0.01" altunitdist="inch" altunit="inch"/>
 <layers>
 <layer number="1" name="Top" color="4" fill="1" visible="no" active="no"/>
@@
 <part name="GND7" library="supply1" deviceset="GND" device=""/>
 <part name="GND34" library="supply1" deviceset="GND" device=""/>
-<part name="C2" library="rcl" deviceset="C-EU" device="C0402" value="0R"/>
 <part name="C15" library="rcl" deviceset="C-EU" device="C0402" value="DNP"/>
 <part name="GND40" library="supply1" deviceset="GND" device=""/>
@@
 <text x="304.8" y="398.78" size="6.4516" layer="94">Spartan IO Banks</text>
 <text x="456.565" y="29.845" size="5.08" layer="94">FPGA / POWER / RF</text>
-<text x="320.675" y="128.27" size="2.54" layer="94">50 ohm lines</text>
 <text x="136.525" y="118.745" size="2.54" layer="97">Spartan 6 Bypass - VCCAUX</text>
 <text x="136.525" y="95.885" size="2.54" layer="97">Spartan 6 Bypass - VCCINT</text>
@@
 <instance part="GND18" gate="1" x="320.675" y="133.35"/>
 <instance part="J1" gate="G$1" x="269.875" y="132.08" rot="MR0"/>
-<instance part="ANT1" gate="G$1" x="264.795" y="175.26"/>
+<instance part="ANT1" gate="G$1" x="264.795" y="176.53"/>
 <instance part="R2" gate="G$1" x="334.645" y="110.49" smashed="yes">
 <attribute name="NAME" x="330.835" y="111.9886" size="1.778" layer="95"/>
@@
 <instance part="GND7" gate="1" x="253.365" y="158.75"/>
 <instance part="GND34" gate="1" x="274.955" y="158.75"/>
-<instance part="C2" gate="G$1" x="339.09" y="167.005" smashed="yes" rot="R270">
-<attribute name="NAME" x="335.534" y="172.466" size="1.778" layer="95"/>
-<attribute name="VALUE" x="335.534" y="169.926" size="1.778" layer="96"/>
-</instance>
 <instance part="C15" gate="G$1" x="304.8" y="161.925" smashed="yes" rot="R180">
 <attribute name="NAME" x="307.594" y="162.306" size="1.778" layer="95"/>
@@
 <wire x1="264.795" y1="161.29" x2="264.795" y2="167.005" width="0.1524" layer="91"/>
 <pinref part="C16" gate="G$1" pin="2"/>
-<wire x1="264.795" y1="167.005" x2="264.795" y2="170.18" width="0.1524" layer="91"/>
+<wire x1="264.795" y1="167.005" x2="264.795" y2="171.45" width="0.1524" layer="91"/>
 <wire x1="288.925" y1="167.005" x2="264.795" y2="167.005" width="0.1524" layer="91"/>
 <junction x="264.795" y="167.005"/>
@@
 <label x="394.335" y="27.305" size="1.778" layer="95"/>
 <wire x1="419.735" y1="28.575" x2="410.845" y2="28.575" width="0.1524" layer="91"/>
-</segment>
-</net>
-<net name="N$29" class="0">
-<segment>
-<wire x1="349.25" y1="167.005" x2="349.25" y2="130.81" width="0.1524" layer="91"/>
-<wire x1="349.25" y1="130.81" x2="353.06" y2="130.81" width="0.1524" layer="91"/>
-<pinref part="U10" gate="_ANA" pin="LNA_IN1"/>
-<pinref part="C2" gate="G$1" pin="1"/>
-<wire x1="349.25" y1="167.005" x2="341.63" y2="167.005" width="0.1524" layer="91"/>
 </segment>
 </net>
@@
 <pinref part="C59" gate="G$1" pin="2"/>
 <wire x1="320.04" y1="167.005" x2="325.12" y2="167.005" width="0.1524" layer="91"/>
-<pinref part="C2" gate="G$1" pin="2"/>
-<wire x1="325.12" y1="167.005" x2="334.01" y2="167.005" width="0.1524" layer="91"/>
+<wire x1="325.12" y1="167.005" x2="349.25" y2="167.005" width="0.1524" layer="91"/>
 <junction x="325.12" y="167.005"/>
-</segment>
-</net>
+<wire x1="349.25" y1="167.005" x2="349.25" y2="130.81" width="0.1524" layer="91"/>
+<wire x1="349.25" y1="130.81" x2="353.06" y2="130.81" width="0.1524" layer="91"/>
+<pinref part="U10" gate="_ANA" pin="LNA_IN1"/>
+</segment>
+</net>

Commit message: Working on the layout
Parts:
- removed ANT1: GPS_PATCH_ANTENNA, joby_robotics:GPS_PATCH_ANTENNA
- removed J3: SMA, joby_robotics:SMA
- added U5: SMA_PATCH, joby_robotics:SMA_PATCH
- J1: value SMA -> SMA_EDGE; device joby_robotics:SMA -> swift-nav:SMA_EDGE
Connections:
- removed net N$45: ANT1.P$1, C16.2, J3.1
- new net 3: J1.2, J1.3
- new net 4: U5.4, U5.5
- new net 5: J1.4, J1.5
- new net N$14: C16.2, U5.1
- net GND: now also U5.2, U5.3; no longer J1.2, J1.3, J1.4, J1.5, J3.2, J3.3, J3.4, J3.5
