File: v2.3/swift-nav.sch (EAGLE design)
At the start: 150 parts, among them J1 SMA_EDGE, J6 ZX62-B-5PA, Q1 IRLML6401, U1 6SLX9FTG256, U10 MAX2769, U12 PT7M8206B33TA5EX, U13 M25PX80, U2 LTC3407A_DFN, U3 STM32-M-64-LQFP, U4 7Q-16.368MBG-T, U5 SMA_PATCH_SMDGND, U6 93LC56BT-I/OT, U7 FT232HQ, U8 B4050, U9 XC2401, X3 FPGA DEBUG, X4 NX5032GA-12M, X5 CONN_5-2

Commit message: Gettin 'er done
Parts:
- L1: value 29nH -> 29nH / DNP
Other:
- moved on the sheet: C16, L4, L5
Changed lines of the file:
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@@
 <part name="C12" library="pel_dipol_comp" deviceset="CAPACITOR" device="-0402" value="100pF"/>
 <part name="C13" library="pel_dipol_comp" deviceset="CAPACITOR" device="-0402" value="0.47uF"/>
-<part name="L1" library="pel_dipol_comp" deviceset="INDUCTOR" device="-0402" value="29nH"/>
+<part name="L1" library="pel_dipol_comp" deviceset="INDUCTOR" device="-0402" value="29nH / DNP"/>
 <part name="L3" library="pel_dipol_comp" deviceset="INDUCTOR" device="-0402" value="29nH"/>
 <part name="R12" library="pel_dipol_comp" deviceset="RESISTOR" device="-0402" value="10k"/>
@@
 </instance>
 <instance part="U8" gate="G$1" x="187.96" y="129.54"/>
-<instance part="GND40" gate="1" x="86.36" y="203.2"/>
+<instance part="GND40" gate="1" x="88.9" y="203.2"/>
 <instance part="U4" gate="U$1" x="119.38" y="147.32"/>
 <instance part="U5" gate="G$1" x="22.86" y="223.52"/>
@@
 <instance part="FRAME4" gate="G$1" x="0" y="0"/>
 <instance part="FRAME4" gate="G$2" x="325.12" y="0"/>
-<instance part="C16" gate="G$1" x="76.2" y="218.44" smashed="yes" rot="R90">
-<attribute name="NAME" x="78.74" y="223.52" size="1.778" layer="95"/>
-<attribute name="VALUE" x="78.74" y="220.98" size="1.778" layer="96"/>
+<instance part="C16" gate="G$1" x="78.74" y="218.44" smashed="yes" rot="R90">
+<attribute name="NAME" x="81.28" y="223.52" size="1.778" layer="95"/>
+<attribute name="VALUE" x="81.28" y="220.98" size="1.778" layer="96"/>
 </instance>
 <instance part="U9" gate="U1" x="119.38" y="218.44"/>
@@
 </instance>
 <instance part="GND84" gate="1" x="83.82" y="22.86"/>
-<instance part="L4" gate="G$1" x="96.52" y="218.44" smashed="yes" rot="R90">
-<attribute name="NAME" x="93.98" y="223.52" size="1.778" layer="95"/>
-<attribute name="VALUE" x="93.98" y="220.98" size="1.778" layer="96"/>
-</instance>
-<instance part="L5" gate="G$1" x="86.36" y="210.82" smashed="yes" rot="R180">
-<attribute name="NAME" x="88.9" y="210.82" size="1.778" layer="95"/>
-<attribute name="VALUE" x="88.9" y="208.28" size="1.778" layer="96"/>
+<instance part="L4" gate="G$1" x="99.06" y="218.44" smashed="yes" rot="R90">
+<attribute name="NAME" x="96.52" y="223.52" size="1.778" layer="95"/>
+<attribute name="VALUE" x="96.52" y="220.98" size="1.778" layer="96"/>
+</instance>
+<instance part="L5" gate="G$1" x="88.9" y="210.82" smashed="yes" rot="R180">
+<attribute name="NAME" x="91.44" y="210.82" size="1.778" layer="95"/>
+<attribute name="VALUE" x="91.44" y="208.28" size="1.778" layer="96"/>
 </instance>
 <instance part="GND62" gate="1" x="48.26" y="177.8"/>
@@
 <segment>
 <pinref part="U5" gate="G$1" pin="1"/>
-<wire x1="73.66" y1="218.44" x2="68.58" y2="218.44" width="0.1524" layer="91"/>
+<wire x1="76.2" y1="218.44" x2="68.58" y2="218.44" width="0.1524" layer="91"/>
 <wire x1="68.58" y1="218.44" x2="25.4" y2="218.44" width="0.1524" layer="91"/>
 <wire x1="68.58" y1="210.82" x2="68.58" y2="218.44" width="0.1524" layer="91"/>
@@
 <segment>
 <pinref part="C16" gate="G$1" pin="2"/>
-<wire x1="81.28" y1="218.44" x2="86.36" y2="218.44" width="0.1524" layer="91"/>
-<wire x1="86.36" y1="218.44" x2="91.44" y2="218.44" width="0.1524" layer="91"/>
-<wire x1="86.36" y1="215.9" x2="86.36" y2="218.44" width="0.1524" layer="91"/>
-<junction x="86.36" y="218.44"/>
+<wire x1="83.82" y1="218.44" x2="88.9" y2="218.44" width="0.1524" layer="91"/>
+<wire x1="88.9" y1="218.44" x2="93.98" y2="218.44" width="0.1524" layer="91"/>
+<wire x1="88.9" y1="215.9" x2="88.9" y2="218.44" width="0.1524" layer="91"/>
+<junction x="88.9" y="218.44"/>
 <pinref part="L4" gate="G$1" pin="1"/>
 <pinref part="L5" gate="G$1" pin="2"/>
@@
 <segment>
 <pinref part="U9" gate="U1" pin="RFIN"/>
-<wire x1="101.6" y1="218.44" x2="104.14" y2="218.44" width="0.1524" layer="91"/>
 <pinref part="L4" gate="G$1" pin="2"/>
 </segment>

Commit message: Gettin' urr dunn
Connections:
- removed net N$1: X3.12
- net DEBUG0: now also U1B3.IO_L32N_M3DQ15_3; no longer U1B3.IO_L36N_M3DQ9_3
- net DEBUG1: now also U1B3.IO_L34N_M3UDQSN_3; no longer U1B3.IO_L38N_M3DQ3_3
- net DEBUG2: now also U1B3.IO_L35N_M3DQ11_3; no longer U1B3.IO_L40N_M3DQ7_3
- net DEBUG3: now also U1B3.IO_L36N_M3DQ9_3; no longer U1B3.IO_L41N_GCLK26_M3DQ5_3
- net DEBUG4: now also U1B3.IO_L38N_M3DQ3_3; no longer U1B3.IO_L49N_M3A2_3
- net DEBUG5: now also U1B3.IO_L44N_GCLK20_M3A6_3; no longer U1B3.IO_L50P_M3WE_3
- net DEBUG6: now also U1B3.IO_L41N_GCLK26_M3DQ5_3; no longer U1B3.IO_L50N_M3BA2_3
- net DEBUG7: now also U1B3.IO_L46N_M3CLKN_3
- net DEBUG8: now also U1B3.IO_L49N_M3A2_3
- net DEBUG9: now also U1B3.IO_L50P_M3WE_3
- net V+: now also X3.12
Other:
- moved on the sheet: U1B3
Changed lines of the file:
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@@
 <setting verticaltext="up"/>
 </settings>
-<grid distance="0.1" unitdist="inch" unit="inch" style="lines" multiple="1" display="no" altdistance="0.01" altunitdist="inch" altunit="inch"/>
+<grid distance="0.1" unitdist="inch" unit="inch" style="lines" multiple="1" display="yes" altdistance="0.01" altunitdist="inch" altunit="inch"/>
 <layers>
 <layer number="1" name="Top" color="4" fill="1" visible="no" active="no"/>
@@
 <part name="C36" library="pel_dipol_comp" deviceset="CAPACITOR" device="-0402" value="100pF"/>
 <part name="C41" library="pel_dipol_comp" deviceset="CAPACITOR" device="-0402" value="0.47uF"/>
+<part name="P+3" library="supply1" deviceset="V+" device=""/>
 </parts>
 <sheets>
@@
 <instance part="U1" gate="B1" x="134.62" y="165.1"/>
 <instance part="U1" gate="B2" x="220.98" y="163.83"/>
-<instance part="U1" gate="B3" x="368.3" y="163.83"/>
+<instance part="U1" gate="B3" x="368.3" y="165.1"/>
 <instance part="U1" gate="BNA" x="73.66" y="39.37"/>
 <instance part="GND35" gate="1" x="238.76" y="19.05"/>
@@
 <instance part="VCC19" gate="G$1" x="46.99" y="226.06"/>
 <instance part="VCC20" gate="G$1" x="147.32" y="243.84"/>
-<instance part="VCC21" gate="G$1" x="378.46" y="242.57"/>
+<instance part="VCC21" gate="G$1" x="378.46" y="243.84"/>
 <instance part="GND28" gate="1" x="257.048" y="12.446"/>
 <instance part="FRAME1" gate="G$1" x="0" y="0"/>
@@
 </segment>
 <segment>
-<wire x1="373.38" y1="227.33" x2="378.46" y2="227.33" width="0.1524" layer="91"/>
-<wire x1="378.46" y1="227.33" x2="378.46" y2="229.87" width="0.1524" layer="91"/>
-<wire x1="378.46" y1="229.87" x2="378.46" y2="232.41" width="0.1524" layer="91"/>
-<wire x1="378.46" y1="232.41" x2="378.46" y2="234.95" width="0.1524" layer="91"/>
-<wire x1="378.46" y1="234.95" x2="378.46" y2="237.49" width="0.1524" layer="91"/>
-<wire x1="378.46" y1="237.49" x2="378.46" y2="240.03" width="0.1524" layer="91"/>
-<wire x1="373.38" y1="229.87" x2="378.46" y2="229.87" width="0.1524" layer="91"/>
-<wire x1="373.38" y1="232.41" x2="378.46" y2="232.41" width="0.1524" layer="91"/>
-<wire x1="373.38" y1="234.95" x2="378.46" y2="234.95" width="0.1524" layer="91"/>
-<wire x1="373.38" y1="237.49" x2="378.46" y2="237.49" width="0.1524" layer="91"/>
-<junction x="378.46" y="229.87"/>
-<junction x="378.46" y="232.41"/>
-<junction x="378.46" y="234.95"/>
-<junction x="378.46" y="237.49"/>
+<wire x1="373.38" y1="228.6" x2="378.46" y2="228.6" width="0.1524" layer="91"/>
+<wire x1="378.46" y1="228.6" x2="378.46" y2="231.14" width="0.1524" layer="91"/>
+<wire x1="378.46" y1="231.14" x2="378.46" y2="233.68" width="0.1524" layer="91"/>
+<wire x1="378.46" y1="233.68" x2="378.46" y2="236.22" width="0.1524" layer="91"/>
+<wire x1="378.46" y1="236.22" x2="378.46" y2="238.76" width="0.1524" layer="91"/>
+<wire x1="378.46" y1="238.76" x2="378.46" y2="241.3" width="0.1524" layer="91"/>
+<wire x1="373.38" y1="231.14" x2="378.46" y2="231.14" width="0.1524" layer="91"/>
+<wire x1="373.38" y1="233.68" x2="378.46" y2="233.68" width="0.1524" layer="91"/>
+<wire x1="373.38" y1="236.22" x2="378.46" y2="236.22" width="0.1524" layer="91"/>
+<wire x1="373.38" y1="238.76" x2="378.46" y2="238.76" width="0.1524" layer="91"/>
+<junction x="378.46" y="231.14"/>
+<junction x="378.46" y="233.68"/>
+<junction x="378.46" y="236.22"/>
+<junction x="378.46" y="238.76"/>
 <pinref part="U1" gate="B3" pin="VCCO_3@4"/>
 <pinref part="VCC21" gate="G$1" pin="VCCIO"/>
@@
 <net name="DEBUG6" class="0">
 <segment>
-<wire x1="373.38" y1="123.19" x2="382.651" y2="123.19" width="0.1524" layer="91"/>
-<label x="383.159" y="123.19" size="1.778" layer="95"/>
-<pinref part="U1" gate="B3" pin="IO_L50N_M3BA2_3"/>
-</segment>
-</net>
-<net name="DEBUG5" class="0">
-<segment>
-<wire x1="373.38" y1="120.65" x2="382.651" y2="120.65" width="0.1524" layer="91"/>
-<label x="383.286" y="120.65" size="1.778" layer="95"/>
-<pinref part="U1" gate="B3" pin="IO_L50P_M3WE_3"/>
-</segment>
-</net>
-<net name="DEBUG4" class="0">
-<segment>
-<wire x1="373.38" y1="128.27" x2="382.651" y2="128.27" width="0.1524" layer="91"/>
-<label x="383.286" y="128.27" size="1.778" layer="95"/>
-<pinref part="U1" gate="B3" pin="IO_L49N_M3A2_3"/>
-</segment>
-</net>
-<net name="DEBUG3" class="0">
-<segment>
-<wire x1="373.38" y1="168.91" x2="382.651" y2="168.91" width="0.1524" layer="91"/>
-<label x="383.54" y="168.91" size="1.778" layer="95"/>
+<wire x1="373.38" y1="170.18" x2="386.08" y2="170.18" width="0.1524" layer="91"/>
+<label x="386.08" y="170.18" size="1.778" layer="95"/>
 <pinref part="U1" gate="B3" pin="IO_L41N_GCLK26_M3DQ5_3"/>
 </segment>
 </net>
-<net name="DEBUG2" class="0">
-<segment>
-<wire x1="373.38" y1="173.99" x2="382.651" y2="173.99" width="0.1524" layer="91"/>
-<label x="383.54" y="173.99" size="1.778" layer="95"/>
-<pinref part="U1" gate="B3" pin="IO_L40N_M3DQ7_3"/>
-</segment>
-</net>
-<net name="DEBUG1" class="0">
-<segment>
-<wire x1="373.38" y1="184.15" x2="382.651" y2="184.15" width="0.1524" layer="91"/>
-<pinref part="U1" gate="B3" pin="IO_L38N_M3DQ3_3"/>
-<label x="383.54" y="184.15" size="1.778" layer="95"/>
-</segment>
-</net>
-<net name="DEBUG0" class="0">
+<net name="DEBUG5" class="0">
 <segment>
-<label x="383.286" y="194.31" size="1.778" layer="95"/>
-<wire x1="373.38" y1="194.31" x2="382.651" y2="194.31" width="0.1524" layer="91"/>
-<pinref part="U1" gate="B3" pin="IO_L36N_M3DQ9_3"/>
+<wire x1="373.38" y1="154.94" x2="386.08" y2="154.94" width="0.1524" layer="91"/>
+<label x="386.08" y="154.94" size="1.778" layer="95"/>
+<pinref part="U1" gate="B3" pin="IO_L44N_GCLK20_M3A6_3"/>
 </segment>
 </net>
@@
 </segment>
 </net>
+<net name="DEBUG9" class="0">
+<segment>
+<wire x1="373.38" y1="121.92" x2="386.08" y2="121.92" width="0.1524" layer="91"/>
+<label x="386.08" y="121.92" size="1.778" layer="95"/>
+<pinref part="U1" gate="B3" pin="IO_L50P_M3WE_3"/>
+</segment>
+</net>
+<net name="DEBUG8" class="0">
+<segment>
+<wire x1="373.38" y1="129.54" x2="386.08" y2="129.54" width="0.1524" layer="91"/>
+<label x="386.08" y="129.54" size="1.778" layer="95"/>
+<pinref part="U1" gate="B3" pin="IO_L49N_M3A2_3"/>
+</segment>
+</net>
+<net name="DEBUG7" class="0">
+<segment>
+<wire x1="373.38" y1="144.78" x2="386.08" y2="144.78" width="0.1524" layer="91"/>
+<label x="386.08" y="144.78" size="1.778" layer="95"/>
+<pinref part="U1" gate="B3" pin="IO_L46N_M3CLKN_3"/>
+</segment>
+</net>
+<net name="DEBUG4" class="0">
+<segment>
+<wire x1="373.38" y1="185.42" x2="386.08" y2="185.42" width="0.1524" layer="91"/>
+<label x="386.08" y="185.42" size="1.778" layer="95"/>
+<pinref part="U1" gate="B3" pin="IO_L38N_M3DQ3_3"/>
+</segment>
+</net>
+<net name="DEBUG3" class="0">
+<segment>
+<wire x1="373.38" y1="195.58" x2="386.08" y2="195.58" width="0.1524" layer="91"/>
+<label x="386.08" y="195.58" size="1.778" layer="95"/>
+<pinref part="U1" gate="B3" pin="IO_L36N_M3DQ9_3"/>
+</segment>
+</net>
+<net name="DEBUG2" class="0">
+<segment>
+<wire x1="373.38" y1="200.66" x2="386.08" y2="200.66" width="0.1524" layer="91"/>
+<label x="386.08" y="200.66" size="1.778" layer="95"/>
+<pinref part="U1" gate="B3" pin="IO_L35N_M3DQ11_3"/>
+</segment>
+</net>
+<net name="DEBUG1" class="0">
+<segment>
+<wire x1="373.38" y1="205.74" x2="386.08" y2="205.74" width="0.1524" layer="91"/>
+<label x="386.08" y="205.74" size="1.778" layer="95"/>
+<pinref part="U1" gate="B3" pin="IO_L34N_M3UDQSN_3"/>
+</segment>
+</net>
+<net name="DEBUG0" class="0">
+<segment>
+<wire x1="373.38" y1="215.9" x2="386.08" y2="215.9" width="0.1524" layer="91"/>
+<label x="386.08" y="215.9" size="1.778" layer="95"/>
+<pinref part="U1" gate="B3" pin="IO_L32N_M3DQ15_3"/>
+</segment>
+</net>
 </nets>
 </sheet>
@@
 <attribute name="VALUE" x="137.16" y="198.12" size="5.08" layer="91" rot="R180"/>
 </instance>
+<instance part="P+3" gate="1" x="114.3" y="185.42" smashed="yes">
+<attribute name="VALUE" x="113.03" y="187.96" size="1.778" layer="96"/>
+</instance>
 </instances>
 <busses>
@@
 <wire x1="43.18" y1="86.36" x2="33.02" y2="86.36" width="0.1524" layer="91"/>
 </segment>
+<segment>
+<wire x1="114.3" y1="152.4" x2="114.3" y2="182.88" width="0.1524" layer="91"/>
+<pinref part="X3" gate="G$1" pin="12"/>
+<wire x1="106.68" y1="152.4" x2="114.3" y2="152.4" width="0.1524" layer="91"/>
+<pinref part="P+3" gate="1" pin="V+"/>
+</segment>
 </net>
 <net name="V_USB" class="0">
@@
 </segment>
 </net>
-<net name="N$1" class="0">
-<segment>
-<wire x1="114.3" y1="152.4" x2="114.3" y2="185.42" width="0.1524" layer="91"/>
-<pinref part="X3" gate="G$1" pin="12"/>
-<wire x1="106.68" y1="152.4" x2="114.3" y2="152.4" width="0.1524" layer="91"/>
-</segment>
-</net>

Commit message: Finished moving stuff around, routing, and DRC. Need to look at soldermask.
Parts:
- added C43, C46, C80, C81: 0.47uF, pel_dipol_comp:CAPACITOR-0402
- added C78: 4.7uF, pel_dipol_comp:CAPACITOR-0603
Connections:
- net GND: now also C43.2, C46.2, C78.2, C80.2, C81.2
- net VCCINT: now also C43.1, C46.1, C78.1, C80.1, C81.1
Other:
- moved on the sheet: C10, C17, C24, C28, C29, C30, C31
Changed lines of the file:
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@@
 <setting verticaltext="up"/>
 </settings>
-<grid distance="0.1" unitdist="inch" unit="inch" style="lines" multiple="1" display="yes" altdistance="0.01" altunitdist="inch" altunit="inch"/>
+<grid distance="0.1" unitdist="inch" unit="inch" style="lines" multiple="1" display="no" altdistance="0.01" altunitdist="inch" altunit="inch"/>
 <layers>
 <layer number="1" name="Top" color="4" fill="1" visible="no" active="no"/>
@@
 <part name="C41" library="pel_dipol_comp" deviceset="CAPACITOR" device="-0402" value="0.47uF"/>
 <part name="P+3" library="supply1" deviceset="V+" device=""/>
+<part name="C43" library="pel_dipol_comp" deviceset="CAPACITOR" device="-0402" value="0.47uF"/>
+<part name="C46" library="pel_dipol_comp" deviceset="CAPACITOR" device="-0402" value="0.47uF"/>
+<part name="C78" library="pel_dipol_comp" deviceset="CAPACITOR" device="-0603" value="4.7uF"/>
+<part name="C80" library="pel_dipol_comp" deviceset="CAPACITOR" device="-0402" value="0.47uF"/>
+<part name="C81" library="pel_dipol_comp" deviceset="CAPACITOR" device="-0402" value="0.47uF"/>
 </parts>
 <sheets>
@@
 <plain>
 <text x="180.34" y="185.42" size="2.54" layer="97">Spartan 6 Bypass - VCCAUX</text>
-<text x="187.96" y="152.4" size="2.54" layer="97">Spartan 6 Bypass - VCCINT</text>
+<text x="172.72" y="152.4" size="2.54" layer="97">Spartan 6 Bypass - VCCINT</text>
 <text x="198.12" y="86.36" size="2.54" layer="97">Spartan 6 Bypass - Bank 3</text>
 <text x="147.32" y="121.92" size="2.54" layer="97">Spartan 6 Bypass - Bank 0</text>
@@
 <instance part="C22" gate="G$1" x="190.5" y="180.34"/>
 <instance part="C23" gate="G$1" x="203.2" y="180.34"/>
-<instance part="C28" gate="G$1" x="182.88" y="147.32"/>
-<instance part="C29" gate="G$1" x="193.04" y="147.32"/>
-<instance part="C30" gate="G$1" x="203.2" y="147.32"/>
-<instance part="C31" gate="G$1" x="213.36" y="147.32"/>
-<instance part="GND24" gate="1" x="226.06" y="137.16"/>
+<instance part="C28" gate="G$1" x="167.64" y="147.32"/>
+<instance part="C29" gate="G$1" x="177.8" y="147.32"/>
+<instance part="C30" gate="G$1" x="187.96" y="147.32"/>
+<instance part="C31" gate="G$1" x="198.12" y="147.32"/>
+<instance part="GND24" gate="1" x="248.92" y="137.16"/>
 <instance part="GND25" gate="1" x="215.9" y="170.18"/>
 <instance part="U1" gate="BGND" x="43.18" y="124.46"/>
@@
 <instance part="VCC5" gate="G$1" x="177.8" y="187.96"/>
 <instance part="VCC6" gate="G$1" x="124.46" y="142.24"/>
-<instance part="VCC7" gate="G$1" x="182.88" y="154.94"/>
+<instance part="VCC7" gate="G$1" x="137.16" y="154.94"/>
 <instance part="C60" gate="G$1" x="213.36" y="71.12"/>
 <instance part="C62" gate="G$1" x="223.52" y="71.12"/>
@@
 <instance part="C87" gate="G$1" x="203.2" y="71.12"/>
 <instance part="C21" gate="G$1" x="215.9" y="180.34"/>
-<instance part="C24" gate="G$1" x="226.06" y="147.32"/>
-<instance part="C10" gate="G$1" x="172.72" y="147.32"/>
-<instance part="C17" gate="G$1" x="162.56" y="147.32"/>
+<instance part="C24" gate="G$1" x="248.92" y="147.32"/>
+<instance part="C10" gate="G$1" x="157.48" y="147.32"/>
+<instance part="C17" gate="G$1" x="147.32" y="147.32"/>
 <instance part="C25" gate="G$1" x="203.2" y="106.68"/>
 <instance part="C26" gate="G$1" x="160.02" y="71.12"/>
 <instance part="FRAME3" gate="G$1" x="0" y="0"/>
 <instance part="FRAME3" gate="G$2" x="172.72" y="0"/>
+<instance part="C43" gate="G$1" x="208.28" y="147.32"/>
+<instance part="C46" gate="G$1" x="218.44" y="147.32"/>
+<instance part="C78" gate="G$1" x="137.16" y="147.32"/>
+<instance part="C80" gate="G$1" x="238.76" y="147.32"/>
+<instance part="C81" gate="G$1" x="228.6" y="147.32"/>
 </instances>
 <busses>
@@
 </segment>
 <segment>
-<wire x1="226.06" y1="139.7" x2="226.06" y2="142.24" width="0.1524" layer="91"/>
-<wire x1="226.06" y1="142.24" x2="213.36" y2="142.24" width="0.1524" layer="91"/>
-<wire x1="213.36" y1="142.24" x2="203.2" y2="142.24" width="0.1524" layer="91"/>
-<wire x1="203.2" y1="142.24" x2="193.04" y2="142.24" width="0.1524" layer="91"/>
-<wire x1="193.04" y1="142.24" x2="182.88" y2="142.24" width="0.1524" layer="91"/>
-<junction x="226.06" y="142.24"/>
-<junction x="193.04" y="142.24"/>
-<junction x="203.2" y="142.24"/>
-<junction x="213.36" y="142.24"/>
+<wire x1="248.92" y1="139.7" x2="248.92" y2="142.24" width="0.1524" layer="91"/>
+<wire x1="248.92" y1="142.24" x2="238.76" y2="142.24" width="0.1524" layer="91"/>
+<wire x1="238.76" y1="142.24" x2="228.6" y2="142.24" width="0.1524" layer="91"/>
+<wire x1="228.6" y1="142.24" x2="218.44" y2="142.24" width="0.1524" layer="91"/>
+<wire x1="218.44" y1="142.24" x2="208.28" y2="142.24" width="0.1524" layer="91"/>
+<wire x1="208.28" y1="142.24" x2="198.12" y2="142.24" width="0.1524" layer="91"/>
+<wire x1="198.12" y1="142.24" x2="187.96" y2="142.24" width="0.1524" layer="91"/>
+<wire x1="187.96" y1="142.24" x2="177.8" y2="142.24" width="0.1524" layer="91"/>
+<wire x1="177.8" y1="142.24" x2="167.64" y2="142.24" width="0.1524" layer="91"/>
+<junction x="248.92" y="142.24"/>
+<junction x="177.8" y="142.24"/>
+<junction x="187.96" y="142.24"/>
+<junction x="198.12" y="142.24"/>
 <pinref part="GND24" gate="1" pin="GND"/>
 <pinref part="C28" gate="G$1" pin="2"/>
@@
 <pinref part="C24" gate="G$1" pin="2"/>
 <pinref part="C10" gate="G$1" pin="2"/>
-<wire x1="182.88" y1="142.24" x2="172.72" y2="142.24" width="0.1524" layer="91"/>
-<junction x="182.88" y="142.24"/>
+<wire x1="167.64" y1="142.24" x2="157.48" y2="142.24" width="0.1524" layer="91"/>
+<junction x="167.64" y="142.24"/>
 <pinref part="C17" gate="G$1" pin="2"/>
-<wire x1="172.72" y1="142.24" x2="162.56" y2="142.24" width="0.1524" layer="91"/>
-<junction x="172.72" y="142.24"/>
+<wire x1="157.48" y1="142.24" x2="147.32" y2="142.24" width="0.1524" layer="91"/>
+<junction x="157.48" y="142.24"/>
+<pinref part="C43" gate="G$1" pin="2"/>
+<junction x="208.28" y="142.24"/>
+<pinref part="C46" gate="G$1" pin="2"/>
+<junction x="218.44" y="142.24"/>
+<pinref part="C78" gate="G$1" pin="2"/>
+<junction x="147.32" y="142.24"/>
+<wire x1="137.16" y1="142.24" x2="147.32" y2="142.24" width="0.1524" layer="91"/>
+<pinref part="C80" gate="G$1" pin="2"/>
+<junction x="238.76" y="142.24"/>
+<pinref part="C81" gate="G$1" pin="2"/>
+<junction x="228.6" y="142.24"/>
 </segment>
 <segment>
@@
 </segment>
 <segment>
-<wire x1="182.88" y1="152.4" x2="182.88" y2="149.86" width="0.1524" layer="91"/>
-<wire x1="182.88" y1="149.86" x2="193.04" y2="149.86" width="0.1524" layer="91"/>
-<wire x1="193.04" y1="149.86" x2="203.2" y2="149.86" width="0.1524" layer="91"/>
-<wire x1="203.2" y1="149.86" x2="213.36" y2="149.86" width="0.1524" layer="91"/>
-<wire x1="213.36" y1="149.86" x2="226.06" y2="149.86" width="0.1524" layer="91"/>
-<junction x="182.88" y="149.86"/>
-<junction x="193.04" y="149.86"/>
-<junction x="203.2" y="149.86"/>
-<junction x="213.36" y="149.86"/>
+<wire x1="167.64" y1="149.86" x2="177.8" y2="149.86" width="0.1524" layer="91"/>
+<wire x1="177.8" y1="149.86" x2="187.96" y2="149.86" width="0.1524" layer="91"/>
+<wire x1="187.96" y1="149.86" x2="198.12" y2="149.86" width="0.1524" layer="91"/>
+<wire x1="198.12" y1="149.86" x2="208.28" y2="149.86" width="0.1524" layer="91"/>
+<junction x="167.64" y="149.86"/>
+<junction x="177.8" y="149.86"/>
+<junction x="187.96" y="149.86"/>
+<junction x="198.12" y="149.86"/>
 <pinref part="C28" gate="G$1" pin="1"/>
 <pinref part="C29" gate="G$1" pin="1"/>
 <pinref part="C30" gate="G$1" pin="1"/>
 <pinref part="C31" gate="G$1" pin="1"/>
+<pinref part="C24" gate="G$1" pin="1"/>
+<pinref part="C10" gate="G$1" pin="1"/>
+<wire x1="208.28" y1="149.86" x2="218.44" y2="149.86" width="0.1524" layer="91"/>
+<wire x1="218.44" y1="149.86" x2="228.6" y2="149.86" width="0.1524" layer="91"/>
+<wire x1="228.6" y1="149.86" x2="238.76" y2="149.86" width="0.1524" layer="91"/>
+<wire x1="238.76" y1="149.86" x2="248.92" y2="149.86" width="0.1524" layer="91"/>
+<wire x1="157.48" y1="149.86" x2="167.64" y2="149.86" width="0.1524" layer="91"/>
+<pinref part="C17" gate="G$1" pin="1"/>
+<wire x1="157.48" y1="149.86" x2="147.32" y2="149.86" width="0.1524" layer="91"/>
+<junction x="157.48" y="149.86"/>
+<junction x="147.32" y="149.86"/>
+<pinref part="C43" gate="G$1" pin="1"/>
+<junction x="208.28" y="149.86"/>
+<pinref part="C46" gate="G$1" pin="1"/>
+<junction x="218.44" y="149.86"/>
+<pinref part="C78" gate="G$1" pin="1"/>
+<wire x1="147.32" y1="149.86" x2="137.16" y2="149.86" width="0.1524" layer="91"/>
 <pinref part="VCC7" gate="G$1" pin="VCCINT"/>
-<pinref part="C24" gate="G$1" pin="1"/>
-<pinref part="C17" gate="G$1" pin="1"/>
-<pinref part="C10" gate="G$1" pin="1"/>
-<wire x1="162.56" y1="149.86" x2="172.72" y2="149.86" width="0.1524" layer="91"/>
-<wire x1="172.72" y1="149.86" x2="182.88" y2="149.86" width="0.1524" layer="91"/>
-<junction x="172.72" y="149.86"/>
-</segment>
-</net>
+<wire x1="137.16" y1="152.4" x2="137.16" y2="149.86" width="0.1524" layer="91"/>
+<junction x="137.16" y="149.86"/>
+<pinref part="C80" gate="G$1" pin="1"/>
+<junction x="238.76" y="149.86"/>
+<pinref part="C81" gate="G$1" pin="1"/>
+<junction x="228.6" y="149.86"/>
+</segment>
+</net>
