File: piksi/piksi.brd (EAGLE design)
At the start: 53 x 53 mm, 157 parts, among them J1 SMA_EDGE, J6 ZX62-B-5PA, Q1 IRLML6401, U1 6SLX9FTG256, U10 MAX2769, U12 PT7M8206B33TA5EX, U13 M25PX80, U2 LTC3407A_DFN, U3 STM32-M-64-LQFP, U4 7Q-16.368MBG-T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

Commit message: Changed L1 inductor value to DNP
Parts:
- L1: value 27nH / DNP -> DNP
Changed lines of the file:
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@@
 <element name="C12" library="pel_dipol_comp" package="0402-CAP" value="100pF" x="48.514" y="24.1427" rot="R90"/>
 <element name="C13" library="pel_dipol_comp" package="0402-CAP" value="0.47uF" x="47.0281" y="24.7904"/>
-<element name="L1" library="pel_dipol_comp" package="0402-IND" value="27nH / DNP" x="31.6484" y="26.8097" rot="R90"/>
+<element name="L1" library="pel_dipol_comp" package="0402-IND" value="DNP" x="31.6484" y="26.8097" rot="R90"/>
 <element name="L3" library="pel_dipol_comp" package="0402-IND" value="3.3nH" x="48.26" y="26.6319" rot="R270"/>
 <element name="R12" library="pel_dipol_comp" package="0402-RES" value="10k" x="35.2298" y="32.5882" rot="R180"/>
