File: piksi/piksi.sch (EAGLE design)
At the start: 156 parts, among them J1 SMA_EDGE, J6 ZX62-B-5PA, Q1 IRLML6401, U1 6SLX9FTG256, U10 MAX2769, U12 PT7M8206B33TA5EX, U13 M25PX80, U2 LTC3407A_DFN, U3 STM32-M-64-LQFP, U4 7Q-16.368MBG-T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

Commit message: Changed frame, description, and added copyright/license notice for sheet 2
Other:
- note added: "FPGA IO Banks / JTAG / Flash"
- note removed: "FPGA IO / JTAG / FLASH"
- moved on the sheet: C48, R13, R14, R15, R16, R17, R18, U1B0, U1B1, U1B2, U1B3, U1BNA

Commit message: Changed frame, description, and added copyright/license notice for sheet 1
Other:
- note removed: "2.3.1"
- moved on the sheet: B1, C27, C32, C33, C51, C52, C53, C54, C55, C66, C82, LED1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
